Commit message: camera distortion fix

File: urc_gazebo/urdf/drone.xacro (robot description, xacro)
@@ -75,5 +75,124 @@
 		<xacro:default_inertial mass="${0.01}" p="${0}" ix_value="${0}" iy_value="${0}" iz_value="${2.4-5}" />
 	</link>
-	<!-- Front-Facing Camera -->
+<!-- ======================================================== -->
+	<link name="plate2">
+		<visual>
+			<origin xyz="0 0 0" rpy="0 0 0" />
+			<geometry>
+				<box size="${0.05} ${0.03} ${0.005}" />
+			</geometry>
+			<material name="blue" />
+		</visual>
+		<collision>
+			<origin xyz="0 0 0" rpy="0 0 0" />
+			<geometry>
+				<box size="${0.05} ${0.03} ${0.005}" />
+			</geometry>
+		</collision>
+		<xacro:default_inertial mass="${0.001}" p="${0}" ix_value="${0}" iy_value="${0}" iz_value="${8.1666-7}" />
+	</link>
+<!-- ======================================================== -->
+	<link name="cyl1">
+		<visual>
+			<origin xyz="0 0 0" rpy="0 0 0" />
+			<geometry>
+				<cylinder radius="0.016" length="0.02" />
+			</geometry>
+			<material name="golden" />
+		</visual>
+		<collision>
+			<origin xyz="0 0 0" rpy="0 0 0" />
+			<geometry>
+				<cylinder radius="0.016" length="0.02" />
+			</geometry>
+		</collision>
+		<xacro:default_inertial mass="${0.01}" p="${0}" ix_value="${8.95e-6}" iy_value="${8.95e-6}" iz_value="${2.23e-4}" />
+	</link>
+<!-- ======================================================== -->
+	<link name="cyl2">
+		<visual>
+			<origin xyz="0 0 0" rpy="0 0 0" />
+			<geometry>
+				<cylinder radius="0.016" length="0.02" />
+			</geometry>
+			<material name="golden" />
+		</visual>
+		<collision>
+			<origin xyz="0 0 0" rpy="0 0 0" />
+			<geometry>
+				<cylinder radius="0.016" length="0.02" />
+			</geometry>
+		</collision>
+		<xacro:default_inertial mass="${0.01}" p="${0}" ix_value="${8.95e-6}" iy_value="${8.95e-6}" iz_value="${2.23e-4}" />
+	</link>
+<!-- ======================================================== -->
+	<link name="cyl3">
+		<visual>
+			<origin xyz="0 0 0" rpy="0 0 0" />
+			<geometry>
+				<cylinder radius="0.016" length="0.02" />
+			</geometry>
+			<material name="golden" />
+		</visual>
+		<collision>
+			<origin xyz="0 0 0" rpy="0 0 0" />
+			<geometry>
+				<cylinder radius="0.016" length="0.02" />
+			</geometry>
+		</collision>
+		<xacro:default_inertial mass="${0.01}" p="${0}" ix_value="${8.95e-6}" iy_value="${8.95e-6}" iz_value="${2.23e-4}" />
+	</link>
+<!-- ======================================================== -->
+	<link name="cyl4">
+		<visual>
+			<origin xyz="0 0 0" rpy="0 0 0" />
+			<geometry>
+				<cylinder radius="0.016" length="0.02" />
+			</geometry>
+			<material name="golden" />
+		</visual>
+		<collision>
+			<origin xyz="0 0 0" rpy="0 0 0" />
+			<geometry>
+				<cylinder radius="0.016" length="0.02" />
+			</geometry>
+		</collision>
+		<xacro:default_inertial mass="${0.01}" p="${0}" ix_value="${8.95e-6}" iy_value="${8.95e-6}" iz_value="${2.23e-4}" />
+	</link>
+<!-- ======================================================== -->
+	<link name="arduino">
+		<visual>
+			<origin xyz="0 0 0" rpy="0 0 0" />
+			<geometry>
+				<mesh filename="package://fly_bot/meshes/22V10.dae" scale="0.005 0.005 0.005" />
+			</geometry>
+		</visual>
+		<collision>
+			<origin xyz="0 0 0" rpy="0 0 0" />
+			<geometry>
+				<box size="0.1 0.1 0.001" />
+			</geometry>
+		</collision>
+		<xacro:default_inertial mass="${0.05}" p="${0}" ix_value="${0}" iy_value="${0}" iz_value="${8.33333e-5}" />
+	</link>
+<!-- ======================================================== -->
+	<link name="camera_link">
+		<visual>
+			<origin xyz="0 0 0" rpy="0 0 0" />
+			<geometry>
+				<box size="0.01 0.01 0.01" />
+			</geometry>
+			<material name="red" />
+		</visual>
+		<collision>
+			<origin xyz="0 0 0" rpy="0 0 0" />
+			<geometry>
+				<box size="0.01 0.01 0.01" />
+			</geometry>
+		</collision>
+		<xacro:default_inertial mass="${1e-5}" p="${0}" ix_value="${1e-6}" iy_value="${1e-6}" iz_value="${1e-6}" />
+	</link>
+<!-- ======================================================== -->
+<!-- Front-Facing Camera -->
 	<link name="cam/front">
           <visual>
@@ -96,29 +215,4 @@
 	  <child link="cam/front"/>
         </joint>
-	<gazebo reference="cam/front">
-          <sensor name="front_sensor" type="camera">
-            <plugin name="front_sensor" filename="libgazebo_ros_camera.so">
-              <ros>
-                <namespace>/image</namespace>
-                <remapping>~/image_raw:=front_img</remapping>
-                <remapping>~/camera_info:=front_info</remapping>
-              </ros>
-              <initial_orientation_as_reference>false</initial_orientation_as_reference>
-            </plugin>
-            <always_on>true</always_on>
-            <update_rate>100</update_rate>
-            <visualize>true</visualize>
-            <camera name="cam/front">
-              <distortion>
-                <k1>0.1</k1>
-                <k2>0.2</k2>
-                <k3>0.3</k3>
-                <p1>0.4</p1>
-                <p2>0.5</p2>
-                <center>0.5 0.5</center>
-              </distortion>
-             </camera>
-           </sensor>
-        </gazebo>
         <!-- Bottom-Facing Camera -->
         <link name="cam/bottom">
@@ -142,147 +236,4 @@
 	  <child link="cam/bottom"/>
         </joint>
-	<gazebo reference="cam/bottom">
-          <sensor name="bottom_sensor" type="camera">
-            <plugin name="bottom_sensor" filename="libgazebo_ros_camera.so">
-              <ros>
-                <namespace>/image</namespace>
-                <remapping>~/image_raw:=bottom_img</remapping>
-                <remapping>~/camera_info:=bottom_info</remapping>
-              </ros>
-              <initial_orientation_as_reference>false</initial_orientation_as_reference>
-            </plugin>
-            <always_on>true</always_on>
-            <update_rate>100</update_rate>
-            <visualize>true</visualize>
-            <camera name="cam/bottom">
-              <distortion>
-                <k1>0.1</k1>
-                <k2>0.2</k2>
-                <k3>0.3</k3>
-                <p1>0.4</p1>
-                <p2>0.5</p2>
-                <center>0.5 0.5</center>
-              </distortion>
-             </camera>
-           </sensor>
-        </gazebo>
-<!-- ======================================================== -->
-	<link name="plate2">
-		<visual>
-			<origin xyz="0 0 0" rpy="0 0 0" />
-			<geometry>
-				<box size="${0.05} ${0.03} ${0.005}" />
-			</geometry>
-			<material name="blue" />
-		</visual>
-		<collision>
-			<origin xyz="0 0 0" rpy="0 0 0" />
-			<geometry>
-				<box size="${0.05} ${0.03} ${0.005}" />
-			</geometry>
-		</collision>
-		<xacro:default_inertial mass="${0.001}" p="${0}" ix_value="${0}" iy_value="${0}" iz_value="${8.1666-7}" />
-	</link>
-<!-- ======================================================== -->
-	<link name="cyl1">
-		<visual>
-			<origin xyz="0 0 0" rpy="0 0 0" />
-			<geometry>
-				<cylinder radius="0.016" length="0.02" />
-			</geometry>
-			<material name="golden" />
-		</visual>
-		<collision>
-			<origin xyz="0 0 0" rpy="0 0 0" />
-			<geometry>
-				<cylinder radius="0.016" length="0.02" />
-			</geometry>
-		</collision>
-		<xacro:default_inertial mass="${0.01}" p="${0}" ix_value="${8.95e-6}" iy_value="${8.95e-6}" iz_value="${2.23e-4}" />
-	</link>
-<!-- ======================================================== -->
-	<link name="cyl2">
-		<visual>
-			<origin xyz="0 0 0" rpy="0 0 0" />
-			<geometry>
-				<cylinder radius="0.016" length="0.02" />
-			</geometry>
-			<material name="golden" />
-		</visual>
-		<collision>
-			<origin xyz="0 0 0" rpy="0 0 0" />
-			<geometry>
-				<cylinder radius="0.016" length="0.02" />
-			</geometry>
-		</collision>
-		<xacro:default_inertial mass="${0.01}" p="${0}" ix_value="${8.95e-6}" iy_value="${8.95e-6}" iz_value="${2.23e-4}" />
-	</link>
-<!-- ======================================================== -->
-	<link name="cyl3">
-		<visual>
-			<origin xyz="0 0 0" rpy="0 0 0" />
-			<geometry>
-				<cylinder radius="0.016" length="0.02" />
-			</geometry>
-			<material name="golden" />
-		</visual>
-		<collision>
-			<origin xyz="0 0 0" rpy="0 0 0" />
-			<geometry>
-				<cylinder radius="0.016" length="0.02" />
-			</geometry>
-		</collision>
-		<xacro:default_inertial mass="${0.01}" p="${0}" ix_value="${8.95e-6}" iy_value="${8.95e-6}" iz_value="${2.23e-4}" />
-	</link>
-<!-- ======================================================== -->
-	<link name="cyl4">
-		<visual>
-			<origin xyz="0 0 0" rpy="0 0 0" />
-			<geometry>
-				<cylinder radius="0.016" length="0.02" />
-			</geometry>
-			<material name="golden" />
-		</visual>
-		<collision>
-			<origin xyz="0 0 0" rpy="0 0 0" />
-			<geometry>
-				<cylinder radius="0.016" length="0.02" />
-			</geometry>
-		</collision>
-		<xacro:default_inertial mass="${0.01}" p="${0}" ix_value="${8.95e-6}" iy_value="${8.95e-6}" iz_value="${2.23e-4}" />
-	</link>
-<!-- ======================================================== -->
-	<link name="arduino">
-		<visual>
-			<origin xyz="0 0 0" rpy="0 0 0" />
-			<geometry>
-				<mesh filename="package://fly_bot/meshes/22V10.dae" scale="0.005 0.005 0.005" />
-			</geometry>
-		</visual>
-		<collision>
-			<origin xyz="0 0 0" rpy="0 0 0" />
-			<geometry>
-				<box size="0.1 0.1 0.001" />
-			</geometry>
-		</collision>
-		<xacro:default_inertial mass="${0.05}" p="${0}" ix_value="${0}" iy_value="${0}" iz_value="${8.33333e-5}" />
-	</link>
-<!-- ======================================================== -->
-	<link name="camera_link">
-		<visual>
-			<origin xyz="0 0 0" rpy="0 0 0" />
-			<geometry>
-				<box size="0.01 0.01 0.01" />
-			</geometry>
-			<material name="red" />
-		</visual>
-		<collision>
-			<origin xyz="0 0 0" rpy="0 0 0" />
-			<geometry>
-				<box size="0.01 0.01 0.01" />
-			</geometry>
-		</collision>
-		<xacro:default_inertial mass="${1e-5}" p="${0}" ix_value="${1e-6}" iy_value="${1e-6}" iz_value="${1e-6}" />
-	</link>
 <!-- ======================================================== -->
 	<!-- Propellers of the quad: fr, fl, br, bl -->
@@ -497,53 +448,3 @@
 		</actuator>
 	</transmission>
-<gazebo>
-  <sensor type="camera" name="front_sensor">
-          <!-- Set always_on only sensor, not on plugin -->
-          <always_on>0</always_on>
-          <!-- Set update_rate only sensor, not on plugin -->
-          <update_rate>1</update_rate>
-          <!-- Use camera, not camera_triggered -->
-          <plugin name="front_sensor" filename="libgazebo_ros_camera.so">
-            <!-- Change namespace, camera name and topics so:
-                 * Images are published to: /custom_ns/custom_camera/custom_image
-                 * Camera info is published to: /custom_ns/custom_camera/custom_info
-            -->
-            <ros>
-              <namespace>/image</namespace>
-              <argument>~/image_raw:=front_img</argument>
-              <argument>~/camera_info:=front_info</argument>
-            </ros>
-            <!-- Set camera name. If empty, defaults to sensor name (i.e. "sensor_name") -->
-            <camera_name>front_camera</camera_name>
-            <!-- Set TF frame name. If empty, defaults to link name (i.e. "link_name") -->
-            <frame_name>front_tf</frame_name>
-            <hack_baseline>0.07</hack_baseline>
-            <!-- No need to repeat distortion parameters or to set autoDistortion -->
-          </plugin>
-        </sensor>
-  <sensor type="camera" name="bottom_sensor">
-          <!-- Set always_on only sensor, not on plugin -->
-          <always_on>0</always_on>
-          <!-- Set update_rate only sensor, not on plugin -->
-          <update_rate>1</update_rate>
-          <!-- Use camera, not camera_triggered -->
-          <plugin name="bottom_sensor" filename="libgazebo_ros_camera.so">
-            <!-- Change namespace, camera name and topics so:
-                 * Images are published to: /custom_ns/custom_camera/custom_image
-                 * Camera info is published to: /custom_ns/custom_camera/custom_info
-            -->
-            <ros>
-              <namespace>/image</namespace>
-              <argument>~/image_raw:=bottom_img</argument>
-              <argument>~/camera_info:=bottom_info</argument>
-            </ros>
-            <!-- Set camera name. If empty, defaults to sensor name (i.e. "sensor_name") -->
-            <camera_name>bottom_camera</camera_name>
-            <!-- Set TF frame name. If empty, defaults to link name (i.e. "link_name") -->
-            <frame_name>bottom_tf</frame_name>
-            <hack_baseline>0.07</hack_baseline>
-            <!-- No need to repeat distortion parameters or to set autoDistortion -->
-          </plugin>
-        </sensor>
-</gazebo>
 </robot>

Commit message: + gps, +imu(orientation)

File: urc_gazebo/urdf/drone.xacro (robot description, xacro)
@@ -237,4 +237,44 @@
         </joint>
 <!-- ======================================================== -->
+        <link name="gps">
+    	<visual>
+     	 <geometry>
+     	   <box size="0.01 0.01 0.01"/>
+     	 </geometry>
+    	</visual>
+   	<collision>
+          <geometry>
+            <box size="0.01 0.01 0.01"/>
+   	 </geometry>
+        </collision>
+    	<xacro:box_inertia m="0.1" w="0.1" d="0.1" h="0.1"/>
+  	</link>
+   	<joint name="gps_joint" type="fixed">
+		<axis xyz="1 0 0"/>
+		<origin xyz="0 0 0.02"/>
+		<parent link="plate1"/>
+		<child link="gps"/>
+	</joint>
+<!-- ======================================================== -->
+       <link name="imu">
+    	<visual>
+      	<geometry>
+        	<box size="0.01 0.01 0.01"/>
+      	</geometry>
+    	</visual>
+    	<collision>
+      	<geometry>
+       	 <box size="0.01 0.01 0.01"/>
+      	</geometry>
+    	</collision>
+    	<xacro:box_inertia m="0.1" w="0.1" d="0.1" h="0.1"/>
+  	</link>
+  	<joint name="imu_joint" type="fixed">
+		<axis xyz="1 0 0"/>
+		<origin xyz="0 0 -0.02"/>
+		<parent link="plate1"/>
+		<child link="imu"/>
+	</joint>
+<!-- ======================================================== -->
 	<!-- Propellers of the quad: fr, fl, br, bl -->
 	<link name="prop_front_right">
